Commit message: moving to arm64

File: urdf/my_arm.urdf.xacro (robot description, xacro)
@@ -18,4 +18,5 @@
     <inertial>
       <mass value="0.5"/>
+      <origin xyz="0 0 0" rpy="0 0 0"/> <!-- Add origin for clarity, though default is 0 0 0 -->
       <inertia ixx="0.001" ixy="0.0" ixz="0.0" iyy="0.001" iyz="0.0" izz="0.001"/>
     </inertial>
@@ -46,5 +47,6 @@
       <inertial>
         <mass value="0.1"/>
-        <inertia ixx="0.0001" ixy="0.0" ixz="0.0" iyy="0.0001" izz="0.0001"/>
+        <origin xyz="0 0 0" rpy="0 0 0"/> <!-- Add origin for clarity -->
+        <inertia ixx="0.0001" ixy="0.0" ixz="0.0" iyy="0.0001" iyz="0.0" izz="0.0001"/> <!-- Added ixy, ixz, iyz -->
       </inertial>
     </link>
@@ -57,23 +59,4 @@
   <xacro:arm_joint prefix="joint_wrist1" parent_link="link_wrist1" child_link="link_wrist2" origin_xyz="0 0 0.05" origin_rpy="0 0 0" joint_type="revolute"/>
   <xacro:arm_joint prefix="joint_wrist2" parent_link="link_wrist2" child_link="link_gripper" origin_xyz="0 0 0.05" origin_rpy="0 0 0" joint_type="revolute"/>
-  <link name="link_gripper">
-    <visual>
-      <geometry>
-        <box size="0.03 0.03 0.03"/>
-      </geometry>
-      <material name="red">
-        <color rgba="1 0 0 1"/>
-      </material>
-    </visual>
-    <collision>
-      <geometry>
-        <box size="0.03 0.03 0.03"/>
-      </geometry>
-    </collision>
-    <inertial>
-      <mass value="0.05"/>
-      <inertia ixx="0.00001" ixy="0.0" ixz="0.0" iyy="0.00001" izz="0.00001"/>
-    </inertial>
-  </link>
   <!-- ROS 2 Control Hardware Interface -->
   <ros2_control name="ArduinoArmHardware" type="system">
